File: PNIN Technical/PNIN Device V1/PCB Designs/PNIN Device V1/PNIN Device V1.kicad_sch (KiCad schematic)
At the start: 24 parts, among them P1 USB_C_Plug, SW1 RotaryEncoder_Switch, U1 ATmega328P-A, U2 FT232RL, Y1 Crystal

Commit message: update
Parts:
- added C9: 100nf, symbol Device:C
- added J1: Conn_02x04_Odd_Even, symbol Connector_Generic:Conn_02x04_Odd_Even
- added J2: Conn_01x04, symbol Connector_Generic:Conn_01x04
- added J3: Conn_01x08, symbol Connector_Generic:Conn_01x08
- added J4: Conn_01x03, symbol Connector_Generic:Conn_01x03
- added R10: 2K, symbol Device:R
- added R11: 1K, symbol Device:R
- added R12: 10K, symbol Device:R
- added SW2: SW_SPST, symbol Switch:SW_SPST
Connections:
- net +5V: now also J2.2 (Pin_2), J3.1 (Pin_1)
- net A4/SDA: now also J2.4 (Pin_4), J3.4 (Pin_4)
- net A5/SCL: now also J2.3 (Pin_3), J3.3 (Pin_3)
- net D0/RX: now also R1.2; no longer R1.1
- net D1/TX: now also R2.1, R11.1; no longer R2.2
- net GND: now also C9.2, J1.1 (Pin_1), J2.1 (Pin_1), J3.2 (Pin_2), R10.2
- net RX: now also SW2.2 (B); no longer R2.1, U2.1 (TXD)
- net at P1.B5 (VCONN), R6.1: now also P1.A5 (CC), R7.1
- net +3.3V: now reaches U2.17 (3V3OUT)
- net +3.3V: now also C9.1, J1.8 (Pin_8), R12.1
- net TX: no longer names the net of U2.5 (RXD)
- net TX: now also R2.2; no longer R1.2
- new net: R1.1, U2.1 (TXD)
- new net CH_EN: J1.4 (Pin_4), R12.2
- new net D11: J3.8 (Pin_8)
- new net ESP_RESET: J1.6 (Pin_6)
- new net GPIO0: J1.5 (Pin_5)
- new net GPIO1/TX: J1.2 (Pin_2), SW2.1 (A)
- new net GPIO2: J1.3 (Pin_3)
- new net GPIO3/RX: J1.7 (Pin_7), R10.1, R11.2
- no-connect marks 22 -> 24
Other:
- note added: "ESP01"
- note added: "MPU6050 IMU Sensor"
- note added: "OLED Screen"
- moved on the sheet: P1, R1, R2
